File: eda/camera_badge/camera_badge.kicad_sch (KiCad schematic)
At the start: 0 parts

Commit message: eda updates
Parts:
- added DS1: GC9A01 TFT Display, 0_local:GC9A01_TFT, symbol 0_local:GC9A01 TFT Display
- added U1: ESP32-WROOM-32-DEVKIT, 0_local:ESP32_DEVKIT_V1, symbol 0_local:ESP32-WROOM-32-DEVKIT
Connections:
- new net +3.3V: DS1.1 (VCC), U1.1 (3V3)
- new net D16: DS1.5 (DC), U1.6 (GPIO16)
- new net D18: DS1.3 (SCL), U1.9 (GPIO18)
- new net D23: DS1.4 (SDA), U1.15 (GPIO23)
- new net D4: DS1.7 (RST), U1.5 (GPIO4)
- new net D5: DS1.6 (CS), U1.8 (GPIO5)
- new net GND: DS1.2 (GND), U1.2 (GND)
