File: eda/camera_badge/camera_badge.kicad_pcb (KiCad board)
At the start: 2 copper layers, 120.6 x 204.7 mm, 44 parts, among them J1 Battery_Conn, J2 Conn_01x05_Socket, J3 Conn_01x05_Pin, J4 Conn_01x05_Socket, J5 Conn_01x05_Pin, J6 Conn_01x05_Socket, J7 Conn_01x05_Pin, J8 Conn_01x05_Socket, J9 Conn_01x05_Pin, SW1 SW_SPDT_SS12D00G, U1 ESP32-WEMOS-LOLIN32-LITE

Commit message: pcb trace work
Connections:
- D2 pad 2: 14 -> 32
- D5 pad 2: 25 -> 33
- D6 pad 2: 33 -> 25
- D7 pad 2: 32 -> 14
- J4 pad 3: 12 -> 2
- J5 pad 3: 12 -> 2
- J8 pad 3: 2 -> 12
- J9 pad 3: 2 -> 12
- JSAO1 pad 5: 12 -> 2
Routing:
- net 33: track 0.00 -> 142.0 mm
- net 25: track 0.00 -> 114.1 mm
- net GBAT: track 0.00 -> 70.2 mm
- net 2: track 59.9 -> 125.4 mm
- net +3.3V: track 191.5 -> 236.6 mm
- net 32: track 0.00 -> 42.0 mm
- net 0: track 102.4 -> 120.5 mm
- net 12: track 87.2 -> 79.3 mm
- net 14: track 52.5 -> 59.9 mm
- net 15: track 76.1 -> 83.2 mm
